File: pcb/DSKY_alarm.sch (KiCad schematic (older format))
At the start: 87 parts, among them IC3 ATSAMD21E, SW1 reset, U1 AQY232SZ, U10 AQY232SZ, U11 AQY232SZ, U12 AQY232SZ, U13 AQY232SZ, U14 AQY232SZ, U15 AP2112K-3.3, U2 AQY232SZ, U3 AQY232SZ, U4 AQY232SZ, U5 AQY232SZ, U6 AQY232SZ, U7 AQY232SZ, U8 AQY232SZ, X1 USB_MICRO_20329_V2_revised, u9 AQY232SZ

Commit message: Version 4 of the board
Parts:
- added NT1: Net-Tie_2, NetTie:NetTie-2_SMD_Pad0.5mm, symbol Device:Net-Tie_2
- LA11, LA13, LA21, LA22, LA23, LA31, LA32, LA33, LA41, LA42, LA43, LA51, LA52, LA53, LA61, LA62, LA63, LA71, LA72, LA73, LA81, LA82, LA83, LA91, LA92, LA93, LAA1, LAA2, LAA3, LAB1, LAB2, LAB3, LAC1, LAC2, LAC3, LAD1, LAD2, LAD3, LAE1, LAE2, LAE3: footprint Trinket M0 rev D:VCC7216-ND -> Trinket M0 rev D:VCC7265
- LA12: footprint Trinket M0 rev D:VCC7216-ND -> Trinket M0 rev D:VCC7265; symbol Device:Lamp -> Trinket_M0_rev_D-eagle-import:Lamp_VCC_7265
- X1: value USB_MICRO_20329_V2_revised -> Molex 105133 USB; footprint Trinket M0 rev D:4UCONN_20329_V2_revised -> libraries:MOLEX_105133-0001; symbol Trinket_M0_rev_D-eagle-import:USB_MICRO_20329_V2_revised -> DSKY_alarm-rescue:105133-0001-MOLEX-USB
- renumbered u9 to U9
Connections:
- net labels added: GNDD
- net labels removed: +5V
- wire segments 252 -> 256
- no-connect marks 6 -> 8
Other:
- note removed: "VBAT power is connected\ndirectly to lamps."

Commit message: Updated V4 board to a two layer design
Parts:
- removed NT1: Net-Tie_2, NetTie:NetTie-2_SMD_Pad0.5mm, symbol Device:Net-Tie_2
- removed X1: Molex 105133 USB, libraries:MOLEX_105133-0001, symbol DSKY_alarm-rescue:105133-0001-MOLEX-USB
- added J1: 105133-0001-MOLEX-USB, libraries:MOLEX_105133-0001, symbol DSKY_alarm-rescue:105133-0001-MOLEX-USB
- IC3: symbol Trinket_M0_rev_D-eagle-import:ATSAMD21E -> DSKY_alarm-rescue:ATSAMD21E-Trinket_M0_rev_D-eagle-import
- LA11, LA13, LA21, LA22, LA23, LA31, LA32, LA33, LA41, LA42, LA43, LA51, LA52, LA53, LA61, LA62, LA63, LA71, LA72, LA73, LA81, LA82, LA83, LA91, LA92, LA93, LAA1, LAA2, LAA3, LAB1, LAB2, LAB3, LAC1, LAC2, LAC3, LAD1, LAD2, LAD3, LAE1, LAE2, LAE3: footprint Trinket M0 rev D:VCC7265 -> Trinket M0 rev D:VCC7216-ND
- LA12: footprint Trinket M0 rev D:VCC7265 -> Trinket M0 rev D:VCC7216-ND; symbol Trinket_M0_rev_D-eagle-import:Lamp_VCC_7265 -> Device:Lamp
- renumbered U9 to u9
Connections:
- net labels added: +5V
- net labels removed: GNDD
- wire segments 256 -> 254
- no-connect marks 8 -> 5
Other:
- note added: "VBAT power is connected\ndirectly to lamps."
